File: schematics/Power Board/PowerDistributionBoard.sch (EAGLE design)
At the start: 11 parts

Commit message: Final Board Sent for Fabrication
Parts:
- added JP11, JP8: (no value), pinhead:PINHD-1X2
Connections:
- net N$1: now also JP11.1, JP8.1
- net V-IN1: now also JP11.2, JP8.2
Other:
- moved on the sheet: JP1, JP10, JP2, JP3, JP4, JP5, JP6, JP7, JP9, X1-1, X1-2, X2-1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
