File: schematics/Power Board/SensorBoard.brd (EAGLE design)
At the start: 58.4 x 48.3 mm, 11 parts

Commit message: Updated Most Recent PCB's
Changed both directories with the most up to date schematics.
Routing:
- net COMMON-GND: track 111.3 -> 0.00 mm
- net SENSOR-5V+: track 90.3 -> 0.00 mm
- net V-IN: track 53.1 -> 0.00 mm
- net N$1: track 24.4 -> 0.00 mm
- net N$2: track 3.48 -> 0.00 mm
