File: schematics/Power Board/SensorBoard.sch (EAGLE design)
At the start: 11 parts

Commit message: Updated Most Recent PCB's
Changed both directories with the most up to date schematics.
Parts:
- added JP11, JP8: (no value), pinhead:PINHD-1X2
Connections:
- removed net N$2: JP4.2, JP6.1
- removed net V-IN: JP10.1, JP2.1, JP3.1, JP6.2, JP9.1
- new net V-IN1: JP10.1, JP11.2, JP2.1, JP3.1, JP4.2, JP6.2, JP8.2, JP9.1
- net N$1: now also JP11.1, JP6.1, JP8.1
Other:
- moved on the sheet: JP4, JP6
Changed lines of the file:
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@@
 </part>
 <part name="JP4" library="pinhead" library_urn="urn:adsk.eagle:library:325" deviceset="PINHD-1X2" device="">
+<attribute name="CAP2" value=""/>
+</part>
+<part name="JP6" library="pinhead" library_urn="urn:adsk.eagle:library:325" deviceset="PINHD-1X2" device="">
 <attribute name="CAP1" value=""/>
-</part>
-<part name="JP6" library="pinhead" library_urn="urn:adsk.eagle:library:325" deviceset="PINHD-1X2" device="">
-<attribute name="CAP2" value=""/>
 </part>
 <part name="JP1" library="pinhead" library_urn="urn:adsk.eagle:library:325" deviceset="PINHD-1X2" device="">
 <attribute name="ARDUINO_POWER" value=""/>
+</part>
+<part name="JP8" library="pinhead" library_urn="urn:adsk.eagle:library:325" deviceset="PINHD-1X2" device="">
+<attribute name="CAP4" value=""/>
+</part>
+<part name="JP11" library="pinhead" library_urn="urn:adsk.eagle:library:325" deviceset="PINHD-1X2" device="">
+<attribute name="CAP3" value=""/>
 </part>
 </parts>
@@
 <attribute name="PI-GND" x="91.44" y="40.64" size="1.778" layer="96" rot="R180" display="name"/>
 </instance>
-<instance part="JP4" gate="G$1" x="33.02" y="50.8" rot="R90">
-<attribute name="CAP1" x="33.02" y="55.88" size="1.778" layer="96" rot="R180" display="name"/>
-</instance>
-<instance part="JP6" gate="G$1" x="48.26" y="50.8" rot="R90">
-<attribute name="CAP2" x="48.26" y="55.88" size="1.778" layer="96" rot="R180" display="name"/>
+<instance part="JP4" gate="G$1" x="33.02" y="58.42" rot="R90">
+<attribute name="CAP2" x="38.1" y="50.8" size="1.778" layer="96" display="name"/>
+</instance>
+<instance part="JP6" gate="G$1" x="33.02" y="48.26" rot="R90">
+<attribute name="CAP1" x="38.1" y="40.64" size="1.778" layer="96" display="name"/>
 </instance>
 <instance part="JP1" gate="G$1" x="-7.62" y="30.48" rot="R90">
 <attribute name="ARDUINO_POWER" x="-7.62" y="35.56" size="1.778" layer="96" rot="R180" display="name"/>
+</instance>
+<instance part="JP8" gate="G$1" x="33.02" y="78.74" rot="R90">
+<attribute name="CAP4" x="38.1" y="71.12" size="1.778" layer="96" display="name"/>
+</instance>
+<instance part="JP11" gate="G$1" x="33.02" y="68.58" rot="R90">
+<attribute name="CAP3" x="38.1" y="60.96" size="1.778" layer="96" display="name"/>
 </instance>
 </instances>
@@
 </busses>
 <nets>
-<net name="V-IN" class="0">
-<segment>
-<pinref part="JP2" gate="A" pin="1"/>
-<wire x1="68.58" y1="40.64" x2="60.96" y2="40.64" width="0.1524" layer="91"/>
-<junction x="68.58" y="40.64"/>
-<wire x1="68.58" y1="48.26" x2="68.58" y2="40.64" width="0.1524" layer="91"/>
-<pinref part="JP3" gate="A" pin="1"/>
-<wire x1="60.96" y1="40.64" x2="60.96" y2="25.4" width="0.1524" layer="91"/>
-<wire x1="60.96" y1="25.4" x2="68.58" y2="25.4" width="0.1524" layer="91"/>
-<pinref part="JP9" gate="A" pin="1"/>
-<wire x1="60.96" y1="25.4" x2="60.96" y2="10.16" width="0.1524" layer="91"/>
-<wire x1="60.96" y1="10.16" x2="68.58" y2="10.16" width="0.1524" layer="91"/>
-<junction x="60.96" y="25.4"/>
-<pinref part="JP10" gate="A" pin="1"/>
-<wire x1="60.96" y1="10.16" x2="60.96" y2="-5.08" width="0.1524" layer="91"/>
-<wire x1="60.96" y1="-5.08" x2="68.58" y2="-5.08" width="0.1524" layer="91"/>
-<junction x="60.96" y="10.16"/>
-<label x="68.58" y="45.72" size="1.778" layer="95"/>
-<pinref part="JP6" gate="G$1" pin="2"/>
-<wire x1="48.26" y1="48.26" x2="68.58" y2="48.26" width="0.1524" layer="91"/>
-</segment>
-</net>
 <net name="SENSOR-5V+" class="0">
 <segment>
@@
 <segment>
 <pinref part="X1" gate="-1" pin="KL"/>
-<wire x1="17.78" y1="30.48" x2="17.78" y2="48.26" width="0.1524" layer="91"/>
+<wire x1="17.78" y1="30.48" x2="17.78" y2="45.72" width="0.1524" layer="91"/>
 <pinref part="JP4" gate="G$1" pin="1"/>
-<wire x1="17.78" y1="48.26" x2="30.48" y2="48.26" width="0.1524" layer="91"/>
+<wire x1="17.78" y1="45.72" x2="17.78" y2="55.88" width="0.1524" layer="91"/>
+<wire x1="17.78" y1="55.88" x2="30.48" y2="55.88" width="0.1524" layer="91"/>
 <pinref part="JP1" gate="G$1" pin="2"/>
 <wire x1="-7.62" y1="27.94" x2="-5.08" y2="30.48" width="0.1524" layer="91"/>
@@
 <wire x1="-7.62" y1="27.94" x2="-10.16" y2="27.94" width="0.1524" layer="91"/>
 <junction x="-7.62" y="27.94"/>
-</segment>
-</net>
-<net name="N$2" class="0">
-<segment>
+<pinref part="JP6" gate="G$1" pin="1"/>
+<wire x1="17.78" y1="45.72" x2="30.48" y2="45.72" width="0.1524" layer="91"/>
+<junction x="17.78" y="45.72"/>
+<pinref part="JP8" gate="G$1" pin="1"/>
+<wire x1="17.78" y1="76.2" x2="30.48" y2="76.2" width="0.1524" layer="91"/>
+<pinref part="JP11" gate="G$1" pin="1"/>
+<wire x1="17.78" y1="66.04" x2="30.48" y2="66.04" width="0.1524" layer="91"/>
+<wire x1="17.78" y1="55.88" x2="17.78" y2="66.04" width="0.1524" layer="91"/>
+<junction x="17.78" y="55.88"/>
+<wire x1="17.78" y1="66.04" x2="17.78" y2="76.2" width="0.1524" layer="91"/>
+<junction x="17.78" y="66.04"/>
+</segment>
+</net>
+<net name="V-IN1" class="0">
+<segment>
+<pinref part="JP8" gate="G$1" pin="2"/>
+<wire x1="33.02" y1="76.2" x2="68.58" y2="76.2" width="0.1524" layer="91"/>
+<pinref part="JP11" gate="G$1" pin="2"/>
+<wire x1="33.02" y1="66.04" x2="68.58" y2="66.04" width="0.1524" layer="91"/>
+<wire x1="68.58" y1="76.2" x2="68.58" y2="66.04" width="0.1524" layer="91"/>
+<pinref part="JP2" gate="A" pin="1"/>
+<wire x1="68.58" y1="40.64" x2="60.96" y2="40.64" width="0.1524" layer="91"/>
+<junction x="68.58" y="40.64"/>
+<wire x1="68.58" y1="55.88" x2="68.58" y2="45.72" width="0.1524" layer="91"/>
+<pinref part="JP3" gate="A" pin="1"/>
+<wire x1="68.58" y1="45.72" x2="68.58" y2="40.64" width="0.1524" layer="91"/>
+<wire x1="60.96" y1="40.64" x2="60.96" y2="25.4" width="0.1524" layer="91"/>
+<wire x1="60.96" y1="25.4" x2="68.58" y2="25.4" width="0.1524" layer="91"/>
+<pinref part="JP9" gate="A" pin="1"/>
+<wire x1="60.96" y1="25.4" x2="60.96" y2="10.16" width="0.1524" layer="91"/>
+<wire x1="60.96" y1="10.16" x2="68.58" y2="10.16" width="0.1524" layer="91"/>
+<junction x="60.96" y="25.4"/>
+<pinref part="JP10" gate="A" pin="1"/>
+<wire x1="60.96" y1="10.16" x2="60.96" y2="-5.08" width="0.1524" layer="91"/>
+<wire x1="60.96" y1="-5.08" x2="68.58" y2="-5.08" width="0.1524" layer="91"/>
+<junction x="60.96" y="10.16"/>
+<label x="68.58" y="45.72" size="1.778" layer="95"/>
 <pinref part="JP4" gate="G$1" pin="2"/>
-<pinref part="JP6" gate="G$1" pin="1"/>
-<wire x1="33.02" y1="48.26" x2="45.72" y2="48.26" width="0.1524" layer="91"/>
-</segment>
-</net>
+<wire x1="33.02" y1="55.88" x2="68.58" y2="55.88" width="0.1524" layer="91"/>
+<pinref part="JP6" gate="G$1" pin="2"/>
+<wire x1="33.02" y1="45.72" x2="68.58" y2="45.72" width="0.1524" layer="91"/>
+<junction x="68.58" y="45.72"/>
+<wire x1="68.58" y1="66.04" x2="68.58" y2="55.88" width="0.1524" layer="91"/>
+<junction x="68.58" y="66.04"/>
+<junction x="68.58" y="55.88"/>
+</segment>
+</net>
